File: usbC_power_controller.kicad_sch (KiCad schematic)
At the start: 0 parts

Commit message: first prototype of a working sma board
Parts:
- added J1: Conn_Coaxial, Connector_Coaxial:SMA_Molex_73251-2200_Horizontal, symbol Connector:Conn_Coaxial
- added J3: Conn_01x02_Pin, Connector_Molex:Molex_Mini-Fit_Jr_5566-02A_2x01_P4.20mm_Vertical, symbol Connector:Conn_01x02_Pin
- added J4: USB_A_Stacked, Connector_USB:USB_A_Wuerth_61400826021_Horizontal_Stacked, symbol Connector:USB_A_Stacked
- added J5: Conn_01x02_Pin, Connector_PinHeader_2.54mm:PinHeader_1x02_P2.54mm_Vertical, symbol Connector:Conn_01x02_Pin
- added Q1: AO3400A, Package_TO_SOT_SMD:SOT-23, symbol Transistor_FET:AO3400A
- added R1, R3, R5: R, Resistor_THT:R_Axial_DIN0204_L3.6mm_D1.6mm_P5.08mm_Horizontal, symbol Device:R
- added U1: EL817, Package_DIP:DIP-4_W7.62mm_SMDSocket_SmallPads, symbol Isolator:EL817
Connections:
- new net: J1.1 (In), R5.1
- new net: R5.2, U1.1
- new net: Q1.1 (G), R1.2, R3.1
- new net: R1.1, U1.3
- new net GND: J1.2 (Ext), J3.1 (Pin_1), J4.4 (GND1), J4.8 (GND2), J4.9 (Shield), J5.1 (Pin_1), Q1.2 (S), R3.2, U1.2
- new net VCC: J3.2 (Pin_2), J4.1 (VBUS1), J4.5 (VBUS2), J5.2 (Pin_2), U1.4
- new net illumination: J4.3 (D1+), J4.7 (D2+), Q1.3 (D)
- no-connect marks 0 -> 2

Commit message: updated power distribution board
Parts:
- J1: footprint Connector_Coaxial:SMA_Molex_73251-2200_Horizontal -> SMA:SMA_Amphenol_901-143_Horizontal
- J3: footprint Connector_Molex:Molex_Mini-Fit_Jr_5566-02A_2x01_P4.20mm_Vertical -> SMA:Molex_Mini-Fit_Jr_5569-02A2_2x01_P4.20mm_Horizontal
- R1, R3, R5: footprint Resistor_THT:R_Axial_DIN0204_L3.6mm_D1.6mm_P5.08mm_Horizontal -> SMA:R_tht1270_smd3216
Changed lines of the file:
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@@
 			)
 		)
-		(property "Footprint" "Resistor_THT:R_Axial_DIN0204_L3.6mm_D1.6mm_P5.08mm_Horizontal"
+		(property "Footprint" "SMA:R_tht1270_smd3216"
 			(at 155.702 60.96 90)
 			(effects
@@
 			)
 		)
-		(property "Footprint" "Resistor_THT:R_Axial_DIN0204_L3.6mm_D1.6mm_P5.08mm_Horizontal"
+		(property "Footprint" "SMA:R_tht1270_smd3216"
 			(at 181.102 68.58 90)
 			(effects
@@
 			)
 		)
-		(property "Footprint" "Resistor_THT:R_Axial_DIN0204_L3.6mm_D1.6mm_P5.08mm_Horizontal"
+		(property "Footprint" "SMA:R_tht1270_smd3216"
 			(at 179.07 66.548 90)
 			(effects
@@
 			)
 		)
-		(property "Footprint" "Connector_Coaxial:SMA_Molex_73251-2200_Horizontal"
+		(property "Footprint" "SMA:SMA_Amphenol_901-143_Horizontal"
 			(at 139.7 63.5 0)
 			(effects
@@
 			)
 		)
-		(property "Footprint" "Connector_Molex:Molex_Mini-Fit_Jr_5566-02A_2x01_P4.20mm_Vertical"
+		(property "Footprint" "SMA:Molex_Mini-Fit_Jr_5569-02A2_2x01_P4.20mm_Horizontal"
 			(at 187.96 35.56 0)
 			(effects
