File: SMA-interface-pcb.kicad_pcb (KiCad board)
At the start: 2 copper layers, 31.5 x 60 mm, 15 parts, among them J1 Conn_Coaxial, J2 Conn_Coaxial, J3 Conn_01x02_Pin, J4 USB_A_Stacked, J5 Conn_01x02_Pin, Q1 AO3400A, Q2 AO3400A, U1 EL817, U2 EL817

Commit message: updated active buzzer system
Parts:
- removed J2: Conn_Coaxial, Connector_Coaxial:SMA_Amphenol_901-143_Horizontal
- removed Q2: AO3400A, Package_TO_SOT_SMD:SOT-23
- removed R6: R, Resistor_THT:R_Axial_DIN0207_L6.3mm_D2.5mm_P2.54mm_Vertical
- removed U2: EL817, Package_DIP:DIP-4_W7.62mm_SMDSocket_SmallPads
- added J6: Conn_Coaxial, Connector_Coaxial:SMA_Amphenol_901-143_Horizontal, F.Cu at (143.3, 76.8)
- added Q3: AO3400A, Package_TO_SOT_SMD:SOT-23, B.Cu at (158.5, 110.5)
- added R7: R, Resistor_THT:R_Axial_DIN0207_L6.3mm_D2.5mm_P2.54mm_Vertical, F.Cu at (139.3, 84.8)
- added R8: 100, Resistor_THT:R_Axial_DIN0207_L6.3mm_D2.5mm_P2.54mm_Vertical, B.Cu at (157.0, 102.0)
- added R9: 10k, Resistor_THT:R_Axial_DIN0207_L6.3mm_D2.5mm_P2.54mm_Vertical, B.Cu at (153.0, 107.0)
- added RZ1: RP2040-Zero, RP2040:RP2040_Zero_Castellated, F.Cu at (163.5, 84.0)
- added U3: EL817, Package_DIP:DIP-4_W7.62mm_SMDSocket_SmallPads, B.Cu at (145.8, 88.8)
- R1: value R -> 100; moved to B.Cu
- R2, R4: value R -> 10k
- R3: value R -> 10k; moved to B.Cu
- moved J5 39.0 mm to (159.0, 128.0), turned to 90 degrees
- moved R2 20.3 mm to (126.5, 96.0), turned to 0 degrees
- moved J3 19.0 mm to (170.5, 122.3)
- moved R4 11.8 mm to (139.2, 96.8), turned to 0 degrees
- moved R3 11.0 mm to (131.0, 108.0), turned to 0 degrees
- moved Q1 6.87 mm to (139.4, 105.4)
- moved R1 6.86 mm to (131.5, 102.0), turned to 0 degrees
Connections:
- J3 pad 1: GND -> Net-(J3-Pin_1)
- J3 pad 2: VCC -> Net-(J3-Pin_1)
- J4 pad 1: VCC -> Net-(J3-Pin_1)
- J4 pad 5: VCC -> Net-(J3-Pin_1)
- J5 pad 1: GND -> Net-(J3-Pin_1)
- J5 pad 2: VCC -> Net-(J3-Pin_1)
- R1 pad 1: Net-(R1-Pad1) -> Net-(RZ1-GP9)
- R2 pad 1: Net-(J2-In) -> VCC
- R2 pad 2: Net-(R2-Pad2) -> Net-(RZ1-GP0)
- R4 pad 1: Net-(R4-Pad1) -> VCC
- U1 pad 3: Net-(R1-Pad1) -> Net-(RZ1-GP0)
Routing:
- net Net-(J3-Pin_1): track 0.00 -> 95.9 mm
- net GND: track 0.00 -> 64.6 mm
- net VCC: track 73.8 -> 23.8 mm, vias 0 -> 1
- net Net-(RZ1-GP0): track 0.00 -> 36.5 mm
- net Net-(RZ1-GP9): track 0.00 -> 30.2 mm
- net /sound: track 18.9 -> 31.1 mm, vias 0 -> 1
- net Net-(Q3-G): track 0.00 -> 10.9 mm
- net Net-(J2-In): track 10.3 -> 0.00 mm
- net Net-(J6-In): track 0.00 -> 9.61 mm
- net Net-(RZ1-GP10): track 0.00 -> 9.46 mm
- net Net-(R7-Pad2): track 0.00 -> 6.18 mm
- net Net-(R2-Pad2): track 6.10 -> 0.00 mm
- net Net-(RZ1-GP1): track 31.7 -> 26.9 mm
- net Net-(R4-Pad1): track 3.79 -> 0.00 mm
- net Net-(R1-Pad1): track 3.76 -> 0.00 mm
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Other:
- board size 31.5 x 60 mm -> 52 x 60 mm
