File: SMA-interface-pcb.kicad_sch (KiCad schematic)
At the start: 88 parts, among them J1 Conn_01x02_Pin, J10 Conn_01x04_Pin, J11 Conn_01x04_Pin, J12 USB_A_Stacked, J13 Conn_Coaxial, J14 Conn_Coaxial, J15 USB_A_Stacked, J16 Conn_02x03_Odd_Even, J2 Conn_01x02_Pin, J3 Conn_01x02_Pin, J4 Conn_Coaxial, J5 Conn_01x04_Pin, J6 Conn_01x04_Pin, J7 Conn_Coaxial, J8 Conn_Coaxial, J9 Conn_Coaxial, Q1 AO3400A, Q2 AO3400A, Q3 AO3400A, Q4 AO3400A, Q5 AO3400A, Q6 AO3400A, Q7 AO3400A, Q8 AO3400A, U1 74HC7014, U2 TMC2209_SILENTSTEPSTICK, U3 TMC2209_SILENTSTEPSTICK, U4 LM2596T-5, U5 TMC2209_SILENTSTEPSTICK, U6 TMC2209_SILENTSTEPSTICK

Commit message: footprint placement V1
Parts:
- C12, C14, C7, C9: footprint Capacitor_THT:C_Radial_D8.0mm_H11.5mm_P3.50mm -> NeuroACT:CP_Radial_horizontal_D8.0mm_P3.50mm
- C4: footprint Capacitor_THT:CP_Radial_D10.0mm_P5.00mm -> Capacitor_THT:CP_Radial_D8.0mm_P5.00mm
- C5: value 1µF 16V -> 10µF 16V
- D1: value D_TVS -> SMBJ36CA
- D2: value SS56B -> SR5100; footprint Diode_SMD:D_3220_8050Metric_Pad2.65x5.15mm_HandSolder -> Diode_THT:D_DO-201AD_P15.24mm_Horizontal
- J1, J2, J3: footprint Connector_Molex:Molex_Mini-Fit_Jr_5569-02A2_2x01_P4.20mm_Horizontal -> NeuroACT:Molex_Mini-Fit_Jr_5569-02A2_2x01_P4.20mm_Horizontal
- J10, J11, J5, J6: footprint Connector_PinSocket_2.54mm:PinSocket_1x04_P2.54mm_Vertical -> Connector_PinHeader_2.54mm:PinHeader_1x04_P2.54mm_Vertical
- JP1, JP2: footprint Connector_PinSocket_2.54mm:PinSocket_1x03_P2.54mm_Vertical -> Connector_PinHeader_2.54mm:PinHeader_1x03_P2.54mm_Vertical
- U4: footprint Package_TO_SOT_THT:TO-220-5_Vertical -> NeuroACT:TO-220-5_Vertical
- renumbered R28 to R27, R27 to R28
Connections:
- net GND: now also J12.SH (Shield), J15.SH (Shield); no longer J12.9 (Shield), J15.9 (Shield)
- net mot_step_A: now also RZ1.17 (GP26); no longer RZ1.20 (GP29)
- net mot_step_B: now also RZ1.18 (GP27); no longer RZ1.19 (GP28)
- net mot_step_C: now also RZ1.19 (GP28); no longer RZ1.18 (GP27)
- net mot_step_D: now also RZ1.20 (GP29); no longer RZ1.17 (GP26)
